File: Smaller_prototype.kicad_pcb (KiCad board)
At the start: 2 copper layers, 49.5 x 52.6 mm, 77 parts, among them IC1 MAX98357AETE+T, J1 DEBUG, J2 Display_shield, J3 i2s_mic, J4 tp5100, J5 BATTERY, J6 Speaker, J7 Micro_SD_Card, J8 GSB1C411111DS1HR, Q1 BC817, Q2 BC817, SW1 RST, SW3 SW_Push, SW4 SW_Push, SW5 SW_Push, SW6 SW_Push, U2 TPS63000, U3 DFR0299, U4 TPS63000, U6 ESP32-S3-WROOM-1

Commit message: -add some changes to power section and display
Parts:
- removed TP2: P0.29, TestPoint:TestPoint_Pad_D2.0mm
- added C16: 1u, Capacitor_SMD:C_0603_1608Metric_Pad1.08x0.95mm_HandSolder, F.Cu at (78.9, 59.2)
- added C17: 1u, Capacitor_SMD:C_0603_1608Metric_Pad1.08x0.95mm_HandSolder, F.Cu at (78.9, 61.7)
- added C18: 1u, Capacitor_SMD:C_0603_1608Metric_Pad1.08x0.95mm_HandSolder, F.Cu at (78.9, 64.2)
- added C19: 1u, Capacitor_SMD:C_0603_1608Metric_Pad1.08x0.95mm_HandSolder, F.Cu at (78.9, 66.7)
- added C20: 1u, Capacitor_SMD:C_0603_1608Metric_Pad1.08x0.95mm_HandSolder, F.Cu at (78.9, 69.2)
- added C21: 100n, Capacitor_SMD:C_0603_1608Metric_Pad1.08x0.95mm_HandSolder, F.Cu at (29.1, 159.3)
- added C22: 100n, Capacitor_SMD:C_0603_1608Metric_Pad1.08x0.95mm_HandSolder, F.Cu at (29.1, 161.8)
- added C23: 100n, Capacitor_SMD:C_0603_1608Metric_Pad1.08x0.95mm_HandSolder, F.Cu at (195.1, 81.1)
- added IC2: TPS2113ADRBR, lib:SON65P300X300X100-9N-D, F.Cu at (122.9, 157.5)
- added J10: DEBUG, Connector_PinHeader_2.54mm:PinHeader_2x05_P2.54mm_Vertical_SMD, B.Cu at (168.5, 71.5)
- added J11: FPC_40P_LCD_ILI9488, Connector_FFC-FPC:TE_4-1734839-0_1x40-1MP_P0.5mm_Horizontal, F.Cu at (137.8, 79.2)
- added J12: Display, Connector_PinHeader_2.54mm:PinHeader_2x05_P2.54mm_Vertical_SMD, F.Cu at (167.1, 73.6)
- added J9: Conn_02x02_Odd_Even, Connector_PinHeader_2.54mm:PinHeader_2x02_P2.54mm_Vertical_SMD, F.Cu at (152.0, 69.5)
- added R27: DNP, Resistor_SMD:R_0603_1608Metric_Pad0.98x0.95mm_HandSolder, F.Cu at (101.9, 52.4)
- added R28: dnp, Resistor_SMD:R_0603_1608Metric_Pad0.98x0.95mm_HandSolder, F.Cu at (166.5, 64.2)
- added R33: dnp, Resistor_SMD:R_0603_1608Metric_Pad0.98x0.95mm_HandSolder, F.Cu at (169.1, 64.2)
- added R34: R, Resistor_SMD:R_0603_1608Metric_Pad0.98x0.95mm_HandSolder, F.Cu at (113.4, 156.3)
- added R35: R, Resistor_SMD:R_0603_1608Metric_Pad0.98x0.95mm_HandSolder, F.Cu at (113.4, 158.8)
- added R36: R, Resistor_SMD:R_0603_1608Metric_Pad0.98x0.95mm_HandSolder, F.Cu at (113.4, 161.4)
- added R37: R, Resistor_SMD:R_0603_1608Metric_Pad0.98x0.95mm_HandSolder, F.Cu at (129.7, 149.1)
- added R38: R, Resistor_SMD:R_0603_1608Metric_Pad0.98x0.95mm_HandSolder, F.Cu at (129.7, 151.7)
- added R39: 220, Resistor_SMD:R_0603_1608Metric_Pad0.98x0.95mm_HandSolder, F.Cu at (195.1, 83.6)
- added R40: 220, Resistor_SMD:R_0603_1608Metric_Pad0.98x0.95mm_HandSolder, F.Cu at (195.1, 86.1)
- added R41: 220, Resistor_SMD:R_0603_1608Metric_Pad0.98x0.95mm_HandSolder, F.Cu at (195.1, 88.6)
- added SW2: REG_EN, Button_Switch_THT:SW_Slide_SPDT_Angled_CK_OS102011MA1Q, F.Cu at (130.6, 130.3)
- added SW7: SW_Push, Button_Switch_SMD:SW_SPST_B3S-1000, F.Cu at (170.3, 123.2)
- C2, C3: moved to F.Cu
- J1: value DEBUG -> Touch; footprint Connector_PinHeader_2.54mm:PinHeader_2x06_P2.54mm_Vertical_SMD -> Connector_FFC-FPC:TE_0-1734839-6_1x06-1MP_P0.5mm_Horizontal; moved to F.Cu
- J2: value Display_shield -> wireless_charging; footprint Connector_PinHeader_2.54mm:PinHeader_2x13_P2.54mm_Vertical_SMD -> Connector_PinHeader_2.54mm:PinHeader_1x02_P2.54mm_Horizontal
- Q1, Q2, R2, R29, R3, R30: moved to B.Cu
- moved J6 140.4 mm to (19.4, 139.8), turned to 90 degrees
- moved FB5 135.0 mm to (18.4, 166.4), turned to 90 degrees
- moved FB8 132.9 mm to (24.3, 152.1), turned to -90 degrees
- moved C13 126.5 mm to (28.4, 145.0)
- moved FB6 111.7 mm to (26.1, 134.2), turned to 180 degrees
- moved C8 102.0 mm to (208.9, 142.0), turned to 180 degrees
- moved R17 98.0 mm to (206.0, 140.2), turned to -90 degrees
- moved C9 95.6 mm to (209.0, 136.9), turned to 180 degrees
- moved R12 92.6 mm to (206.5, 135.8), turned to -90 degrees
- moved C2 91.5 mm to (237.0, 64.9), turned to 180 degrees
- moved C7 90.3 mm to (209.1, 132.6), turned to -90 degrees
- moved C6 88.6 mm to (206.6, 132.6), turned to -90 degrees
- moved FB7 87.0 mm to (236.4, 68.4), turned to 0 degrees
- moved R16 85.0 mm to (191.1, 139.9), turned to -90 degrees
- moved R22 84.9 mm to (209.1, 128.2), turned to -90 degrees
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Connections:
- C3 pad 1: +3.3V -> GND
- C3 pad 2: GND -> +3.3V
- J1 pad 1: RESET -> +3.3V
- J1 pad 2: +3.3V -> I2C_SDA
- J1 pad 3: /MCU/GPIO_0 -> I2C_SCL
- J1 pad 4: /MCU/GPIO_12/JTAG_TDI -> DISPLAY_TP_IRQ
- J1 pad 5: /MCU/GPIO_1/TXD0 -> DISPLAY_TP_CS
- J1 pad 6: /MCU/GPIO_15/JTAG_TDO -> GND
- J2 pad 1: +3.3V -> VBUS_QI
- J2 pad 2: +5V -> GND
- J4 pad 1: +BATT -> GND
- J4 pad 2: GND -> VBUS
- J4 pad 3: VBUS -> GND
- J4 pad 4: GND -> +BATT
- J8 pad A4B9: VBUS -> VBUS_USB
- J8 pad B4A9: VBUS -> VBUS_USB
- R19 pad 2: Net-(U4-EN) -> REG_EN
- R20 pad 1: Net-(U4-EN) -> REG_EN
- R6 pad 2: Net-(U2-EN) -> REG_EN
- R7 pad 1: Net-(U2-EN) -> REG_EN
- U1 pad 23: unconnected-(U1-P0.01-Pad23) -> I2C_SDA
- U1 pad 39: /MCU/GPIO_3/RXD0 -> /MCU/GPIO_43/TXD0
- U1 pad 40: /MCU/GPIO_2 -> SW5
- U1 pad 41: /MCU/GPIO_1/TXD0 -> /MCU/GPIO_44/RXD0
- U1 pad 7: Net-(U1-P0.29) -> I2C_SCL
- U2 pad 6: Net-(U2-EN) -> REG_EN
- U3 pad 14: D+ -> unconnected-(U3-USB+-Pad14)
- U3 pad 15: D- -> unconnected-(U3-USB--Pad15)
- U4 pad 6: Net-(U4-EN) -> REG_EN
- U6 pad 11: I2S_SCK -> RX
- U6 pad 15: /MCU/GPIO_3/RXD0 -> unconnected-(U6-GPIO3/TOUCH3/ADC1_CH2-Pad15)
- U6 pad 16: SD_CS -> SW4
- U6 pad 21: I2S_WS -> SW5
- U6 pad 23: I2S_SD -> TX
- U6 pad 26: SW4 -> SW3
- U6 pad 31: SW3 -> SD_CS
- U6 pad 36: unconnected-(U6-U0RXD/GPIO44/CLK_OUT2-Pad36) -> /MCU/GPIO_44/RXD0
- U6 pad 37: unconnected-(U6-U0TXD/GPIO43/CLK_OUT1-Pad37) -> /MCU/GPIO_43/TXD0
- U6 pad 38: /MCU/GPIO_2 -> I2S_SD
- U6 pad 39: /MCU/GPIO_1/TXD0 -> I2S_SCK
- U6 pad 4: RX -> I2S_DOUT
- U6 pad 5: TX -> I2S_WS
- U6 pad 8: I2S_DOUT -> I2C_SDA
- U6 pad 9: unconnected-(U6-GPIO16/U0CTS/ADC2_CH5/XTAL_32K_N-Pad9) -> I2C_SCL
Routing:
- net I2C_SCL: track 0.00 -> 114.2 mm, vias 0 -> 4
- net SPI_CLK: track 0.00 -> 94.5 mm, vias 0 -> 2
- net I2C_SDA: track 0.00 -> 92.8 mm, vias 0 -> 1
- net SPI_MOSI: track 0.00 -> 92.8 mm, vias 0 -> 2
- net DISPLAY_DC: track 0.00 -> 87.4 mm, vias 0 -> 6
- net DISPLAY_CS: track 0.00 -> 85.3 mm, vias 0 -> 2
- net DISPLAY_TP_IRQ: track 0.00 -> 71.3 mm, vias 0 -> 3
- net SW3: track 0.00 -> 70.9 mm, vias 0 -> 2
- net DISPLAY_TP_CS: track 0.00 -> 69.1 mm, vias 0 -> 2
- net TX: track 0.00 -> 69.1 mm, vias 0 -> 3
- net I2S_SCK: track 0.00 -> 68.8 mm, vias 0 -> 2
- net /MCU/GPIO_0: track 0.00 -> 62.4 mm, vias 0 -> 4
- net SD_SCK: track 0.00 -> 56.3 mm, vias 0 -> 3
- net DISPLAY_RST: track 0.00 -> 54.8 mm, vias 0 -> 3
- net SW1: track 0.00 -> 52.2 mm, vias 0 -> 2
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Other:
- board size 49.5 x 52.6 mm -> 67.9 x 83.7 mm
- board text added: "For Instructional Use Only."
- board text added: "SOLIDWORKS Educational Product."

Commit message: -enh repin mcu in schematic
Parts:
- added J13: DEBUG_NRF, Connector_PinHeader_2.54mm:PinHeader_2x02_P2.54mm_Vertical_SMD, B.Cu at (162.0, 112.3)
- added SW8: RST, Button_Switch_SMD:SW_SPST_B3S-1000, B.Cu at (160.5, 70.0)
- C15, FB2, R23, R24, R25, R29, R30: moved to F.Cu
- J10: value DEBUG -> DEBUG_ESP; footprint Connector_PinHeader_2.54mm:PinHeader_2x05_P2.54mm_Vertical_SMD -> Connector_PinHeader_2.54mm:PinHeader_2x04_P2.54mm_Vertical_SMD
- moved R29 191.8 mm to (1.68, 0.76), turned to 0 degrees
- moved R30 191.7 mm to (1.68, 3.27), turned to 0 degrees
- moved FB5 145.1 mm to (145.0, 95.5)
- moved J6 133.6 mm to (143.5, 90.5)
- moved FB6 121.3 mm to (141.0, 95.5), turned to 90 degrees
- moved R9 116.3 mm to (165.6, 59.5), turned to 180 degrees
- moved R25 106.8 mm to (154.0, 93.1), turned to -90 degrees
- moved C15 77.7 mm to (153.5, 101.5), turned to 180 degrees
- moved C19 74.5 mm to (127.5, 123.1), turned to -90 degrees
- moved R23 73.4 mm to (151.1, 90.5)
- moved R24 72.2 mm to (151.1, 92.0), turned to 180 degrees
- moved C20 72.2 mm to (149.0, 51.9), turned to -90 degrees
- moved IC1 71.2 mm to (151.0, 95.5), turned to 180 degrees
- moved C13 67.1 mm to (91.1, 121.0)
- moved C21 67.1 mm to (91.8, 135.2)
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Connections:
- J1 pad 5: DISPLAY_TP_CS -> DISPLAY_TP_RST
- J10 pad 3: /MCU/GPIO_0 -> BOOT
- J10 pad 4: /MCU/GPIO_13/JTAG_TCK -> RTS
- J10 pad 5: /MCU/GPIO_43/TXD0 -> DEBUG_UART_TX
- J10 pad 6: /MCU/GPIO_12/JTAG_TDI -> DEBUG_UART_RX
- J10 pad 7: /MCU/GPIO_44/RXD0 -> DTR
- J10 pad 8: RTS -> GND
- J12 pad 1: SPI_MISO -> SPI_MOSI
- J12 pad 2: SPI_CLK -> DISPLAY_DC
- J12 pad 3: SPI_MOSI -> SPI_CLK
- J12 pad 5: DISPLAY_DC -> unconnected-(J12-Pin_5-Pad5)
- J9 pad 1: DISPLAY_TP_CS -> DISPLAY_TP_RST
- Q1 pad 3: /MCU/GPIO_0 -> BOOT
- R31 pad 2: Net-(U1-USB_DM) -> USB_DM_R
- R32 pad 2: Net-(U1-USB_DP) -> USB_DP_R
- R37 pad 1: /MCU/GPIO_14/JTAG_TMS -> /MCU/ADC_CH1
- R38 pad 2: /MCU/GPIO_14/JTAG_TMS -> /MCU/ADC_CH1
- U1 pad 10: SD_MOSI -> TX
- U1 pad 11: SD_MISO -> RX
- U1 pad 12: SD_CS -> DISPLAY_TP_RST
- U1 pad 13: /MCU/GPIO_0 -> DISPLAY_RST
- U1 pad 14: TX -> SW4
- U1 pad 15: Net-(U1-USB_DM) -> USB_DM_R
- U1 pad 16: Net-(U1-USB_DP) -> USB_DP_R
- U1 pad 21: SW2 -> unconnected-(U1-P1.00-Pad21)
- U1 pad 22: DISPLAY_TP_CS -> unconnected-(U1-P0.00-Pad22)
- U1 pad 23: I2C_SDA -> SW2
- U1 pad 24: SW4 -> unconnected-(U1-P1.01-Pad24)
- U1 pad 25: I2S_SCK -> I2S_DOUT
- U1 pad 26: I2S_DOUT -> I2S_SD
- U1 pad 27: DISPLAY_RST -> I2S_WS
- U1 pad 28: I2S_WS -> I2S_SCK
- U1 pad 33: DISPLAY_DC -> SD_SCK
- U1 pad 34: BATT_VOLTAGE -> SD_MOSI
- U1 pad 35: DISPLAY_TP_IRQ -> SD_MISO
- U1 pad 36: SW1 -> SD_CS
- U1 pad 37: SW3 -> DISPLAY_CS
- U1 pad 38: RX -> DISPLAY_DC
- U1 pad 39: /MCU/GPIO_43/TXD0 -> SW1
- U1 pad 4: /MCU/GPIO_12/JTAG_TDI -> SWDIO
- U1 pad 40: SW5 -> SPI_MOSI
- U1 pad 41: /MCU/GPIO_44/RXD0 -> SPI_CLK
- U1 pad 42: DISPLAY_CS -> SW3
- U1 pad 43: SPI_MISO -> DISPLAY_TP_IRQ
- U1 pad 44: SPI_CLK -> I2C_SDA
- U1 pad 45: SPI_MOSI -> I2C_SCL
- U1 pad 5: /MCU/GPIO_13/JTAG_TCK -> SWDCLK
- U1 pad 6: I2S_SD -> SW5
- U1 pad 7: I2C_SCL -> BATT_VOLTAGE
- U1 pad 9: SD_SCK -> /MCU/ADC_CH1
- U6 pad 10: SW2 -> TX
- U6 pad 12: DISPLAY_CS -> SD_CS
- U6 pad 13: Net-(U6-GPIO19/U1RTS/ADC2_CH8/CLK_OUT2/USB_D-) -> USB_DM_R
- U6 pad 14: Net-(U6-GPIO20/U1CTS/ADC2_CH9/CLK_OUT1/USB_D+) -> USB_DP_R
- U6 pad 15: unconnected-(U6-GPIO3/TOUCH3/ADC1_CH2-Pad15) -> SW2
- U6 pad 16: SW4 -> unconnected-(U6-GPIO46-Pad16)
- U6 pad 17: SPI_MISO -> DISPLAY_CS
- U6 pad 19: DISPLAY_RST -> I2S_DOUT
- U6 pad 20: DISPLAY_TP_CS -> I2S_SD
- U6 pad 21: SW5 -> I2S_WS
- U6 pad 22: SW1 -> I2S_SCK
- U6 pad 23: TX -> SD_MISO
- U6 pad 24: DISPLAY_TP_IRQ -> SD_SCK
- U6 pad 25: BATT_VOLTAGE -> SD_MOSI
- U6 pad 26: SW3 -> unconnected-(U6-GPIO45-Pad26)
- U6 pad 27: /MCU/GPIO_0 -> BOOT
- U6 pad 28: SD_MOSI -> unconnected-(U6-SPIIO6/GPIO35/FSPID/SUBSPID-Pad28)
- U6 pad 29: SD_SCK -> unconnected-(U6-SPIIO7/GPIO36/FSPICLK/SUBSPICLK-Pad29)
- U6 pad 30: SD_MISO -> unconnected-(U6-SPIDQS/GPIO37/FSPIQ/SUBSPIQ-Pad30)
- U6 pad 31: SD_CS -> SW1
- U6 pad 32: /MCU/GPIO_13/JTAG_TCK -> DISPLAY_TP_RST
- U6 pad 33: /MCU/GPIO_15/JTAG_TDO -> DISPLAY_RST
- U6 pad 34: /MCU/GPIO_12/JTAG_TDI -> DISPLAY_TP_IRQ
- U6 pad 35: /MCU/GPIO_14/JTAG_TMS -> SW3
- U6 pad 36: /MCU/GPIO_44/RXD0 -> DEBUG_UART_RX
- U6 pad 37: /MCU/GPIO_43/TXD0 -> DEBUG_UART_TX
- U6 pad 38: I2S_SD -> SPI_MOSI
- U6 pad 39: I2S_SCK -> SPI_CLK
- U6 pad 4: I2S_DOUT -> I2C_SDA
- U6 pad 5: I2S_WS -> I2C_SCL
- U6 pad 6: SPI_MOSI -> /MCU/ADC_CH1
- U6 pad 7: SPI_CLK -> BATT_VOLTAGE
- U6 pad 8: I2C_SDA -> SW5
- U6 pad 9: I2C_SCL -> SW4
Routing:
- net SW2: track 0.00 -> 69.3 mm, vias 0 -> 2
- net DISPLAY_TP_CS: track 69.1 -> 0.00 mm, vias 2 -> 0
- net /MCU/GPIO_0: track 62.4 -> 0.00 mm, vias 4 -> 0
- net DISPLAY_TP_RST: track 0.00 -> 54.2 mm, vias 0 -> 1
- net RX: track 0.00 -> 51.3 mm, vias 0 -> 1
- net I2C_SDA: track 92.8 -> 143.5 mm, vias 1 -> 2
- net I2S_SCK: track 68.8 -> 20.8 mm, vias 2 -> 1
- net RESET: track 28.9 -> 73.9 mm, vias 1 -> 2
- net /MCU/GPIO_12/JTAG_TDI: track 43.6 -> 0.00 mm, vias 1 -> 0
- net /MCU/GPIO_13/JTAG_TCK: track 43.0 -> 0.00 mm, vias 1 -> 0
- net SW4: track 0.00 -> 42.5 mm, vias 0 -> 3
- net DISPLAY_RST: track 54.8 -> 90.0 mm
- net BOOT: track 0.00 -> 34.6 mm, vias 0 -> 1
- net SD_SCK: track 56.3 -> 23.8 mm, vias 3 -> 1
- net I2C_SCL: track 114.2 -> 139.8 mm, vias 4 -> 2
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Other:
- board size 67.9 x 83.7 mm -> 72.5 x 108.1 mm

Commit message: -add soft latching circuit, routing mostly done
Parts:
- removed IC2: TPS2113ADRBR, lib:SON65P300X300X100-9N-D
- added IC3: TPS2115ADRBT, lib:SON65P300X300X100-9N-D, F.Cu at (257.2, 123.2)
- added R42: R, Resistor_SMD:R_0603_1608Metric_Pad0.98x0.95mm_HandSolder, F.Cu at (248.4, 144.8)
- added R43: 100k, Resistor_SMD:R_0603_1608Metric_Pad0.98x0.95mm_HandSolder, F.Cu at (240.3, 142.9)
- added R44: 100k, Resistor_SMD:R_0603_1608Metric_Pad0.98x0.95mm_HandSolder, F.Cu at (240.1, 139.6)
- added U5: 74LVC2G74, Package_SO:TSSOP-8_3x3mm_P0.65mm, F.Cu at (245.3, 142.3)
- C1, C10, C2, C21, C22, C23, FB2, FB7, J2, J5, R1, R14, R4, R5: moved to B.Cu
- C12, C4, C9, Q1, Q2, R10, R11, R12, R2, R26, R3, R8: moved to F.Cu
- R29: value 0 -> 10k
- R30: value 0 -> R
- R34: value R -> 0
- R35, R36: value R -> DNP
- moved R29 286.1 mm to (257.2, 129.4), turned to 180 degrees
- moved R30 285.5 mm to (259.0, 127.0)
- moved C16 221.7 mm to (289.2, 129.6), turned to -90 degrees
- moved C21 210.1 mm to (301.0, 115.4)
- moved R14 209.0 mm to (271.0, 110.5), turned to 180 degrees
- moved R27 200.3 mm to (287.4, 127.8), turned to -90 degrees
- moved C10 198.7 mm to (257.4, 109.2), turned to 0 degrees
- moved R8 198.7 mm to (288.2, 142.8), turned to 180 degrees
- moved C14 196.1 mm to (280.8, 109.2), turned to -90 degrees
- moved C17 194.2 mm to (260.4, 130.7), turned to -90 degrees
- moved C1 191.8 mm to (297.3, 113.1), turned to 180 degrees
- moved R26 191.7 mm to (282.6, 143.9), turned to 180 degrees
- moved FB8 190.7 mm to (276.7, 108.5), turned to 0 degrees
- moved R10 188.4 mm to (251.9, 129.0), turned to 90 degrees
- moved R5 187.9 mm to (245.4, 125.7), turned to 0 degrees
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Connections:
- C13 pad 1: +3V3 -> +3.3V
- C18 pad 1: SW3 -> Net-(C18-Pad1)
- FB8 pad 1: +3V3 -> +3.3V
- R11 pad 2: SW3 -> Net-(C18-Pad1)
- R29 pad 1: Net-(U6-GPIO20/U1CTS/ADC2_CH9/CLK_OUT1/USB_D+) -> +3.3V
- R29 pad 2: D+ -> Charger_plugged_in?
- R30 pad 2: D- -> GND
- R34 pad 1: Net-(IC2-VSNS) -> VBUS_USB
- R34 pad 2: GND -> Net-(U1-VBUS)
- R35 pad 1: VBUS_QI -> Net-(C18-Pad1)
- R35 pad 2: Net-(IC2-VSNS) -> SW3
- R36 pad 1: Net-(IC2-ILIM) -> Power_latching_circuit
- R36 pad 2: GND -> Net-(C18-Pad1)
- SW5 pad 2: SW3 -> Net-(C18-Pad1)
- U1 pad 18: unconnected-(U1-VBUS-Pad18) -> Net-(U1-VBUS)
Routing:
- net +3.3V: track 70.9 -> 381.6 mm, vias 1 -> 10
- net +5V: track 7.72 -> 167.5 mm, vias 0 -> 4
- net GND: track 12.5 -> 156.5 mm, vias 1 -> 246
- net Power_latching_circuit: track 0.00 -> 120.3 mm
- net VBUS_USB: track 9.58 -> 95.1 mm
- net +BATT: track 0.00 -> 76.8 mm, vias 0 -> 3
- net Charger_plugged_in?: track 0.00 -> 60.1 mm, vias 0 -> 4
- net REG_EN: track 0.00 -> 52.3 mm, vias 0 -> 2
- net DISPLAY_TP_IRQ: track 48.0 -> 84.5 mm, vias 1 -> 3
- net BATT_VOLTAGE: track 4.90 -> 39.5 mm, vias 1 -> 3
- net DISPLAY_TP_RST: track 54.2 -> 86.2 mm, vias 1 -> 4
- net DISPLAY_DC: track 69.4 -> 99.8 mm, vias 1 -> 2
- net SW2: track 69.3 -> 99.0 mm, vias 2 -> 6
- net SPK2: track 5.86 -> 35.2 mm, vias 0 -> 1
- net SW1: track 37.3 -> 63.2 mm
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- added copper zone on B.Cu, net GND
- added copper zone on F.Cu, net GND

Commit message: -add end revision
Parts:
- removed C23, C3: 100n, Capacitor_SMD:C_0603_1608Metric_Pad1.08x0.95mm_HandSolder
- removed J11: FPC_40P_LCD_ILI9488, Connector_FFC-FPC:TE_4-1734839-0_1x40-1MP_P0.5mm_Horizontal
- removed R39, R40, R41: 220, Resistor_SMD:R_0603_1608Metric_Pad0.98x0.95mm_HandSolder
- added C24: 100n, Capacitor_SMD:C_0603_1608Metric_Pad1.08x0.95mm_HandSolder, F.Cu at (289.5, 133.0)
- added C25: 100n, Capacitor_SMD:C_0603_1608Metric_Pad1.08x0.95mm_HandSolder, B.Cu at (240.5, 93.6)
- added C26: 100n, Capacitor_SMD:C_0603_1608Metric_Pad1.08x0.95mm_HandSolder, B.Cu at (247.8, 80.7)
- added J14: 62684-402100AHLF, lib:62684402100AHLF, F.Cu at (241.2, 85.5)
- added R45: 10k, Resistor_SMD:R_0603_1608Metric_Pad0.98x0.95mm_HandSolder, B.Cu at (248.0, 76.9)
- added R46: 10k, Resistor_SMD:R_0603_1608Metric_Pad0.98x0.95mm_HandSolder, B.Cu at (246.4, 76.9)
- added R47: 10k, Resistor_SMD:R_0603_1608Metric_Pad0.98x0.95mm_HandSolder, B.Cu at (246.2, 80.9)
- added R48: 220, Resistor_SMD:R_0603_1608Metric_Pad0.98x0.95mm_HandSolder, B.Cu at (239.2, 80.3)
- added R49: 220, Resistor_SMD:R_0603_1608Metric_Pad0.98x0.95mm_HandSolder, B.Cu at (235.5, 80.3)
- added R50: 220, Resistor_SMD:R_0603_1608Metric_Pad0.98x0.95mm_HandSolder, B.Cu at (237.4, 80.3)
- added U7: USBLC6-2P6, Package_TO_SOT_SMD:SOT-666, F.Cu at (288.0, 138.6)
- moved R25 1.41 mm to (280.1, 95.7)
- moved R37 1.40 mm to (292.6, 110.3), turned to -90 degrees
- moved R13 1.21 mm to (270.5, 113.3)
- moved R14 1.21 mm to (270.4, 111.6)
- moved U5 0.77 mm to (245.3, 141.5)
- moved R42 0.68 mm to (248.9, 144.3)
- moved SW2 0.47 mm to (248.7, 148.8)
- moved C2 0.38 mm to (302.7, 109.5)
- moved C7 0.25 mm to (263.0, 108.0)
- moved R2 0.25 mm to (301.8, 74.4)
- moved R3 0.12 mm to (301.7, 76.0)
Connections:
- J12 pad 5: unconnected-(J12-Pin_5-Pad5) -> SPI_MISO
- J3 pad 3: I2S_SD -> I2S_WS
- J3 pad 4: I2S_WS -> I2S_SD
- J8 pad A6: D+ -> D+_IN
- J8 pad A7: D- -> D-_IN
- J8 pad B6: D+ -> D+_IN
- J8 pad B7: D- -> D-_IN
- U1 pad 22: unconnected-(U1-P0.00-Pad22) -> SW3
- U1 pad 42: SW3 -> SPI_MISO
- U6 pad 15: SW2 -> SPI_MISO
- U6 pad 16: unconnected-(U6-GPIO46-Pad16) -> SW3
- U6 pad 35: SW3 -> SW2
Routing:
- net GND: track 156.5 -> 279.8 mm, vias 246 -> 238
- net SPI_MISO: track 0.00 -> 107.8 mm, vias 0 -> 6
- net D-: track 58.6 -> 33.3 mm
- net D-_IN: track 0.00 -> 24.3 mm
- net D+: track 51.1 -> 29.6 mm
- net D+_IN: track 0.00 -> 21.0 mm
- net SW2: track 99.0 -> 116.9 mm, vias 6 -> 9
- net SW3: track 51.9 -> 69.1 mm, vias 2 -> 5
- net DISPLAY_DC: track 99.8 -> 85.7 mm, vias 2 -> 5
- net VBUS_USB: track 95.1 -> 108.8 mm
- net DISPLAY_RST: track 91.3 -> 101.8 mm, vias 3 -> 5
- net Net-(J14-Pad6): track 0.00 -> 9.34 mm, vias 0 -> 1
- net SPI_MOSI: track 71.0 -> 79.9 mm, vias 1 -> 3
- net Net-(J11-Pin_34): track 8.31 -> 0.00 mm
- net Net-(J11-Pin_35): track 7.11 -> 0.00 mm
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Other:
- board text added: "+"
- board text added: "+5"
- board text added: "-"
- board text added: "3.3"
- board text added: "BL"
- board text added: "BOOT"
- board text added: "Battery"
- board text added: "CLK"
- board text added: "CS"
- board text added: "Connect as power sw <"
- board text added: "DC"
- board text added: "DFPLAYER ^"
- board text added: "DTR"
- board text added: "Display"
- board text added: "ESP_DEBUG"
- board text added: "G"
- board text added: "GND"
- board text added: "IRQ"
- board text added: "MOSI"
- board text added: "NRF_DEBUG"
- board text added: "RST"
- board text added: "RTS"
- board text added: "RX"
- board text added: "SCL"
- board text added: "SD"
- board text added: "SDA"
- board text added: "SPEAKER"
- board text added: "SW0_PULLUP <"
- board text added: "SW3_PULLUP >"
- board text added: "SW5_PULLUP^"
- board text added: "SWCLK"
- board text added: "SWDIO"
- board text added: "TX"
- board text added: "Touch"
- board text added: "Voice trainer S6 2024"
- board text added: "WS"
- board text added: "Wireless_charger_pad"
- board text added: "^ Connect to GPIO"
- board text added: "^ SW2_PULLUP"
- board text added: "^ SW4_PULLUP"
- board text added: "x"
